Commit message: make obstacles in launch, support multi agent launch, multi_move_test

File: far_ws/src/follow_ahead_rl/urdf/obstacle_urdfs/cylinder.urdf (robot description, URDF)
Before this commit: robot simple_cylinder, 1 links, 0 joints
Links:
- link cylinder_base: geometry collision cylinder length=0.5 radius=0.5; visual cylinder length=0.5 radius=0.5
