Commit message: add halfsize obstacle urdfs, make obstacle urdfs smaller, add function to put obstacles between robots

File: far_ws/src/follow_ahead_rl/urdf/obstacle_urdfs/cylinder_small.urdf (robot description, URDF)
Before this commit: robot simple_cylinder, 1 links, 0 joints
Links:
- link cylinder_base: geometry collision cylinder length=0.125 radius=0.125; visual cylinder length=0.125 radius=0.125
