Commit message: rename obstacle urdf links, tweak between obs placement, teb dynamic obstacle placement

File: far_ws/src/follow_ahead_rl/urdf/obstacle_urdfs/box.urdf (robot description, URDF)
Before this commit: robot simple_box, 1 links, 0 joints
Links:
- removed link box_base
- added link base_link, mass 1.0; collision box size=0.25 0.25 0.25; visual box size=0.25 0.25 0.25

File: far_ws/src/follow_ahead_rl/urdf/obstacle_urdfs/cylinder.urdf (robot description, URDF)
Before this commit: robot simple_cylinder, 1 links, 0 joints
Links:
- removed link cylinder_base
- added link base_link, mass 1.0; collision cylinder length=0.1875 radius=0.1875; visual cylinder length=0.1875 radius=0.1875

File: far_ws/src/follow_ahead_rl/urdf/obstacle_urdfs/cylinder_small.urdf (robot description, URDF)
Before this commit: robot simple_cylinder, 1 links, 0 joints
Links:
- removed link cylinder_base
- added link base_link, mass 1.0; collision cylinder length=0.125 radius=0.125; visual cylinder length=0.125 radius=0.125
